File: co2-uhat.kicad_pcb (KiCad board)
At the start: 2 copper layers, 65 x 30 mm, 23 parts, among them U1 CAT24C32WI-GT3, U2 MH-Z19B

Commit message: co2-uhat.kicad_pcb: Add traces
Add traces to the PCB.

Signed-off-by: Leon Anavi <leon@anavi.org>
Parts:
- moved R2 2.74 mm to (186.9, 86.1), turned to 0 degrees
- moved C1 1.78 mm to (198.1, 86.9)
- moved R3 0.90 mm to (192.8, 86.1), turned to 180 degrees
Routing:
- net +3V3: track 56.9 -> 123.8 mm, vias 0 -> 1
- net +5V: track 0.00 -> 57.1 mm
- net Net-(JP1-Pad1): track 0.00 -> 33.3 mm
- net Net-(R6-Pad2): track 0.00 -> 23.8 mm
- net Net-(R2-Pad2): track 0.00 -> 17.2 mm
- net Net-(R3-Pad2): track 0.00 -> 14.2 mm
- net Net-(D1-Pad2): track 0.00 -> 12.0 mm
- net Net-(R7-Pad2): track 0.00 -> 10.1 mm
- net Net-(D2-Pad2): track 0.00 -> 5.59 mm

Commit message: co2-uhat.kicad_pcb: Move display
Move display and add labels.

Signed-off-by: Leon Anavi <leon@anavi.org>
Parts:
- moved DISPLAY 1.84 mm to (165.4, 102.2)
- renumbered SENS4 to DISPLAY
Routing:
- net GND: track 0.00 -> 5.51 mm, vias 0 -> 1
- net +3V3: track 123.8 -> 125.8 mm
- net Net-(R5-Pad2): track 38.4 -> 40.3 mm
- net Net-(R4-Pad2): track 39.5 -> 40.5 mm
Changed lines of the file:
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@@
       (drillshape 0)
       (scaleselection 1)
-      (outputdirectory "plots/rev11a/")
+      (outputdirectory "plots/rev10/")
     )
   )
@@
     (property "Sheetname" "")
     (attr smd)
-    (fp_text reference "R3" (at 0 -1.9) (layer "F.SilkS")
+    (fp_text reference "R3" (at 0 1.636) (layer "F.SilkS")
       (effects (font (size 0.8 0.8) (thickness 0.1)))
     )
@@
     (property "Sheetname" "")
     (attr smd)
-    (fp_text reference "R5" (at -0.05 1.6) (layer "F.SilkS")
+    (fp_text reference "R5" (at 0.006 1.476) (layer "F.SilkS")
       (effects (font (size 0.8 0.8) (thickness 0.1)))
     )
@@
   )
   (footprint "Pin_Headers:Pin_Header_Straight_1x04" (layer "F.Cu")
-    (at 165.608 100.33 -90)
+    (at 165.395 102.16 -90)
     (descr "Through hole pin header")
     (tags "pin header")
@@
     (property "Sheetname" "")
     (attr through_hole)
-    (fp_text reference "SENS4" (at 0.1 -2.5 90) (layer "F.SilkS")
+    (fp_text reference "DISPLAY" (at 0 -2.745 90) (layer "F.SilkS")
       (effects (font (size 0.7 0.7) (thickness 0.1)))
     )
@@
     (property "Sheetname" "")
     (attr smd)
-    (fp_text reference "R4" (at -0.1 1.55) (layer "F.SilkS")
+    (fp_text reference "R4" (at -0.012 -1.506) (layer "F.SilkS")
       (effects (font (size 0.8 0.8) (thickness 0.1)))
     )
@@
     (property "Sheetname" "")
     (attr through_hole)
-    (fp_text reference "U2" (at -23.368 4.572) (layer "F.SilkS")
-      (effects (font (size 1 1) (thickness 0.15)))
-    )
-    (fp_text value "MH-Z19B" (at -19.05 0.762) (layer "F.Fab")
+    (fp_text reference "U2" (at 0.0153 1.5798) (layer "F.SilkS") hide
+      (effects (font (size 1 1) (thickness 0.15)))
+    )
+    (fp_text value "MH-Z19B" (at -19.05 0.762) (layer "F.Fab") hide
       (effects (font (size 1 1) (thickness 0.15)))
     )
@@
       (net 35 "unconnected-(U2-Pad9)") (pinfunction "PWM") (pintype "passive+no_connect"))
   )
-  (gr_line (start 152 78.46) (end 152 77.46) (layer "B.SilkS") (width 0.2))
   (gr_line (start 210.5011 105.0036) (end 151.5011 105.0036) (layer "Edge.Cuts") (width 0.1))
   (gr_arc (start 151.5011 105.0036) (mid 149.37978 104.12492) (end 148.5011 102.0036) (layer "Edge.Cuts") (width 0.1))
@@
     (effects (font (size 1 1) (thickness 0.15)))
   )
-  (gr_text "SDA SCL GND 3.3V" (at 169.558 92.18 270) (layer "F.SilkS")
-    (effects (font (size 0.8 0.8) (thickness 0.125)))
+  (gr_text "SDA SCL GND 3.3V" (at 169.68 92.09 270) (layer "F.SilkS")
+    (effects (font (size 1 0.8) (thickness 0.125)))
   )
   (gr_text "Rev 1.0 (c) 2023" (at 152.1316 88.6636 90) (layer "F.SilkS")
     (effects (font (size 0.8 0.8) (thickness 0.15)))
   )
-  (gr_text "GND 3.3V SCL SDA" (at 161.6814 103.1748) (layer "F.SilkS")
-    (effects (font (size 0.8 0.8) (thickness 0.125)))
+  (gr_text "GND 3.3V SCL SDA" (at 161.53 99.31) (layer "F.SilkS")
+    (effects (font (size 1 0.8) (thickness 0.125)))
   )
   (gr_text "<" (at 209.9056 83.82 90) (layer "F.SilkS")
@@
   (segment (start 161.998 95.91) (end 167.078 95.91) (width 0.5) (layer "B.Cu") (net 1))
   (segment (start 156.918 95.91) (end 161.998 95.91) (width 0.5) (layer "B.Cu") (net 1))
-  (segment (start 175.0318 102.87) (end 184.9986 92.9032) (width 0.5) (layer "B.Cu") (net 1))
-  (segment (start 160.528 97.38) (end 161.998 95.91) (width 0.5) (layer "B.Cu") (net 1))
-  (segment (start 163.068 102.87) (end 175.0318 102.87) (width 0.5) (layer "B.Cu") (net 1))
-  (segment (start 160.528 100.33) (end 160.528 97.38) (width 0.5) (layer "B.Cu") (net 1))
-  (segment (start 160.528 100.33) (end 163.068 102.87) (width 0.5) (layer "B.Cu") (net 1))
+  (segment (start 160.315 97.593) (end 160.315 102.16) (width 0.5) (layer "B.Cu") (net 1))
+  (segment (start 161.83452 103.67952) (end 160.315 102.16) (width 0.5) (layer "B.Cu") (net 1))
+  (segment (start 161.998 95.91) (end 160.315 97.593) (width 0.5) (layer "B.Cu") (net 1))
   (segment (start 187.3508 90.551) (end 184.9986 92.9032) (width 0.5) (layer "B.Cu") (net 1))
+  (segment (start 174.22228 103.67952) (end 161.83452 103.67952) (width 0.5) (layer "B.Cu") (net 1))
+  (segment (start 184.9986 92.9032) (end 174.22228 103.67952) (width 0.5) (layer "B.Cu") (net 1))
   (segment (start 192.786 90.551) (end 187.3508 90.551) (width 0.5) (layer "B.Cu") (net 1))
+  (via (at 199.49 88.41) (size 0.85) (drill 0.4) (layers "F.Cu" "B.Cu") (net 2))
+  (segment (start 200.5398 89.4598) (end 199.49 88.41) (width 0.5) (layer "B.Cu") (net 2))
+  (segment (start 204.5653 89.4598) (end 200.5398 89.4598) (width 0.5) (layer "B.Cu") (net 2))
   (segment (start 156.464 83.566) (end 155.067 82.169) (width 0.5) (layer "B.Cu") (net 3))
-  (segment (start 155.067 79.043) (end 156.85 77.26) (width 0.5) (layer "B.Cu") (net 3))
+  (segment (start 156.85 77.26) (end 155.067 79.043) (width 0.5) (layer "B.Cu") (net 3))
   (segment (start 204.5653 86.9198) (end 201.2115 83.566) (width 0.5) (layer "B.Cu") (net 3))
   (segment (start 155.067 82.169) (end 155.067 79.043) (width 0.5) (layer "B.Cu") (net 3))
@@
   (segment (start 160.442 86.734) (end 161.998 88.29) (width 0.5) (layer "F.Cu") (net 11))
   (segment (start 160.442 83.566) (end 160.442 86.734) (width 0.5) (layer "F.Cu") (net 11))
-  (segment (start 165.608 100.33) (end 168.656 100.33) (width 0.5) (layer "B.Cu") (net 11))
-  (segment (start 168.656 100.33) (end 171.958 97.028) (width 0.5) (layer "B.Cu") (net 11))
+  (segment (start 165.395 102.16) (end 166.826 102.16) (width 0.5) (layer "B.Cu") (net 11))
   (segment (start 169.316 88.29) (end 167.078 88.29) (width 0.5) (layer "B.Cu") (net 11))
   (segment (start 156.918 88.29) (end 161.998 88.29) (width 0.5) (layer "B.Cu") (net 11))
   (segment (start 171.958 97.028) (end 171.958 90.932) (width 0.5) (layer "B.Cu") (net 11))
+  (segment (start 166.826 102.16) (end 171.958 97.028) (width 0.5) (layer "B.Cu") (net 11))
   (segment (start 171.958 90.932) (end 169.316 88.29) (width 0.5) (layer "B.Cu") (net 11))
   (segment (start 161.998 88.29) (end 167.078 88.29) (width 0.5) (layer "B.Cu") (net 11))
@@
   (segment (start 163.576 89.252) (end 161.998 90.83) (width 0.5) (layer "F.Cu") (net 12))
   (segment (start 168.046 90.83) (end 167.078 90.83) (width 0.5) (layer "B.Cu") (net 12))
+  (segment (start 164.9476 98.298) (end 162.855 100.3906) (width 0.5) (layer "B.Cu") (net 12))
   (segment (start 161.998 90.83) (end 167.078 90.83) (width 0.5) (layer "B.Cu") (net 12))
   (segment (start 156.918 90.83) (end 161.998 90.83) (width 0.5) (layer "B.Cu") (net 12))
+  (segment (start 162.855 100.3906) (end 162.855 102.16) (width 0.5) (layer "B.Cu") (net 12))
   (segment (start 164.9476 98.298) (end 168.402 98.298) (width 0.5) (layer "B.Cu") (net 12))
   (segment (start 168.402 98.298) (end 169.672 97.028) (width 0.5) (layer "B.Cu") (net 12))
-  (segment (start 163.068 100.33) (end 163.068 100.1776) (width 0.5) (layer "B.Cu") (net 12))
   (segment (start 169.672 97.028) (end 169.672 92.456) (width 0.5) (layer "B.Cu") (net 12))
   (segment (start 169.672 92.456) (end 168.046 90.83) (width 0.5) (layer "B.Cu") (net 12))
-  (segment (start 163.068 100.1776) (end 164.9476 98.298) (width 0.5) (layer "B.Cu") (net 12))
   (segment (start 169.4615 83.566) (end 169.164 83.566) (width 0.5) (layer "F.Cu") (net 14))
   (segment (start 168.402 83.566) (end 169.164 83.566) (width 0.254) (layer "F.Cu") (net 14))
