File: co2-uhat.kicad_pcb (KiCad board)
At the start: 2 copper layers, 65 x 30 mm, 23 parts, among them U1 CAT24C32WI-GT3, U2 MH-Z19B

Commit message: co2-uhat.kicad_pcb: Adjust labels
Adjust labels on the front silkscreen and fabrication layer.

Signed-off-by: Leon Anavi <leon@anavi.org>
Parts:
- D1: value LED -> KP-3216EC
- D2: value LED -> KP-3216SGC
Other:
- board text added: "3.3V GND SCL SDA"
- board text removed: "SDA SCL GND 3.3V"
Changed lines of the file:
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@@
       (drillshape 0)
       (scaleselection 1)
-      (outputdirectory "plots/rev10/")
+      (outputdirectory "plots/rev10-bg/")
     )
   )
@@
       (effects (font (size 0.8 0.8) (thickness 0.15)))
     )
-    (fp_text value "LED" (at -0.05 -2 90) (layer "F.Fab")
+    (fp_text value "KP-3216EC" (at -0.05 -2 90) (layer "F.Fab")
       (effects (font (size 0.6 0.6) (thickness 0.15)))
     )
@@
       (effects (font (size 0.8 0.8) (thickness 0.15)))
     )
-    (fp_text value "LED" (at -0.1 -1.95 90) (layer "F.Fab")
+    (fp_text value "KP-3216SGC" (at -0.1 -1.95 90) (layer "F.Fab")
       (effects (font (size 0.6 0.6) (thickness 0.15)))
     )
@@
     (effects (font (size 1 1) (thickness 0.15)))
   )
-  (gr_text "SDA SCL GND 3.3V" (at 169.68 92.09 270) (layer "F.SilkS")
+  (gr_text "3.3V GND SCL SDA" (at 169.73 92.18 90) (layer "F.SilkS")
     (effects (font (size 1 0.8) (thickness 0.125)))
   )
